File: NFCC.kicad_sch (KiCad schematic)
At the start: 67 parts, among them SW5 SW_Push, SW6 SW_SPDT, U10 IIS2MDCTR, U11 24CW1280T-I/OT, U12 BMI088, U7 BMP581, U8 W25N01GVZEIG, U9 PCA9685PW

Commit message: Add files via upload
Parts:
- added D1: SD103AWS, Package_SON:WSON-8-1EP_6x5mm_P1.27mm_EP3.4x4mm, symbol Device:D_Schottky
- added FB1: FerriteBead_Small, symbol Device:FerriteBead_Small
- added J1, J2: USB_B_Micro, Package_DFN_QFN:WQFN-16-1EP_3x3mm_P0.5mm_EP1.75x1.75mm, symbol Connector:USB_B_Micro
- added JP1: SolderJumper_2_Open, Package_SON:WSON-8-1EP_6x5mm_P1.27mm_EP3.4x4mm, symbol Jumper:SolderJumper_2_Open
- added R51, R52: 22, symbol Device:R
- added R53: 560, symbol Device:R
Connections:
- net +5V: now also FB1.2
- net GND: now also J1.5 (GND), J1.SH (Shield), J2.5 (GND), J2.SH (Shield)
- net USB_DM: now also R52.2
- net USB_DP: now also R51.2
- net USB_VBUS: now also JP1.2 (B)
- net DEBUG_TX: now reaches NFCC2.53 (PB14)
- net DEBUG_RX: now reaches NFCC2.54 (PB15)
- net USB_ID: now reaches NFCC2.69 (PA10)
- net USB_ID: now also R53.2
- new net: J1.4 (ID), R53.1
- new net: D1.2 (A), J1.1 (VBUS), JP1.1 (A)
- new net: J1.2 (D-), R52.1
- new net: J1.3 (D+), R51.1
- new net: D1.1 (K), FB1.1
Other:
- note added: "USB Programming"
- moved on the sheet: LED13, LED14, LED15, LED16, LED17, LED18, R35, R36, R37, R39, R40, R41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

Commit message: Add files via upload
Parts:
- added C23, C24: 10u, Package_SO:TSSOP-28_4.4x9.7mm_P0.65mm, symbol Device:C
- added C57, C58, C59, C61: 100n, symbol Device:C
- added C60: 10u, symbol Device:C
- added C62, C63: 22u, symbol Device:C
- added D2: SD103AWS, Package_SON:WSON-8-1EP_6x5mm_P1.27mm_EP3.4x4mm, symbol Device:D_Schottky
- added D3, D4: G, Package_SO:SOIC-8_3.9x4.9mm_P1.27mm, symbol Device:LED
- added FB2: FerriteBead_Small, symbol Device:FerriteBead_Small
- added J3: LiPo Battery, symbol Connector_Generic:Conn_01x02
- added L1: 4.7u, Package_TO_SOT_SMD:SOT-23-6, symbol Device:L
- added R1: 100k, Package_DIP:DIP-8_W7.62mm, symbol Device:R
- added R2: 47k, Package_DIP:DIP-8_W7.62mm, symbol Device:R
- added R3: 52.3k, Package_DIP:DIP-8_W7.62mm, symbol Device:R
- added R54: 560, symbol Device:R
- added R55: 240, symbol Device:R
- added R6, R7: 10k, Package_DIP:DIP-8_W7.62mm, symbol Device:R
- added U1: CH330N, Package_SO:SOIC-8_3.9x4.9mm_P1.27mm, symbol Interface_USB:CH330N
- added U2: TPS54302, Package_TO_SOT_SMD:SOT-23-6, symbol Regulator_Switching:TPS54302
- added U3: LD39200PU33R, SON_DFN6_3X3_STM, symbol 2026-09-15_06-05-24:LD39200PU33R
Connections:
- net +3.3V: now also C24.1, D4.2 (A), U3.1 (OUT), U3.2 (ADJ/SENSE)
- net +5V: now also C23.1, C62.1, C63.1, FB2.2, L1.2, R3.2, U3.5 (EN), U3.6 (IN)
- net BAT_SENSE: now also C59.1, R1.2, R2.1
- net DEBUG_RX: now also U1.6 (TXD)
- net DEBUG_TX: now also U1.7 (RXD)
- net GND: now also C23.2, C24.2, C57.2, C58.2, C59.2, C60.2, C62.2, C63.2, J3.1 (Pin_1), R2.2, R54.1, R55.1, R6.1, U1.3 (GND), U2.1 (GND), U3.3 (GND), U3.7 (GND)
- net at J2.1 (VBUS): now also C58.1, D2.2 (A), D3.2 (A), U1.5 (VCC)
- net at J2.2 (D-): now also U1.2 (UD-)
- net at J2.3 (D+): now also U1.1 (UD+)
- net TELEX_RX renamed TELEM_RX
- new net: D2.1 (K), FB2.1
- new net: D3.1 (K), R54.2
- new net: R7.1, U2.3 (VIN)
- new net: C61.2, L1.1, U2.2 (SW)
- new net: R3.1, R6.2, U2.4 (FB)
- new net: C61.1, U2.6 (BOOT)
- new net: C57.1, U1.8 (V3)
- new net: D4.1 (K), R55.2
- new net VBAT: C60.1, J3.2 (Pin_2), R1.1, R7.2, U2.5 (EN)
- no-connect marks 66 -> 68
Other:
- note added: "3.3V Regulator"
- note added: "5V Buck Converter"
- note added: "LiPo Battery Input"
- note added: "USB Debug"
- moved on the sheet: C12, C16, C18, C19, C51, C52, C53, C54, C55, C56, HSE3, J2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

Commit message: Add files via upload
Parts:
- C12: footprint Package_SO:TSSOP-28_4.4x9.7mm_P0.65mm -> NFCC:C_0603_1608Metric__C12
- C13: footprint Package_SO:TSSOP-28_4.4x9.7mm_P0.65mm -> NFCC:C_0603_1608Metric__C13
- C14: footprint Package_SO:TSSOP-28_4.4x9.7mm_P0.65mm -> NFCC:C_0603_1608Metric__C14
- C15: footprint Package_SO:TSSOP-28_4.4x9.7mm_P0.65mm -> NFCC:C_0603_1608Metric__C15
- C16: footprint Package_SO:TSSOP-28_4.4x9.7mm_P0.65mm -> NFCC:C_0603_1608Metric__C16
- C17: footprint Package_SO:TSSOP-28_4.4x9.7mm_P0.65mm -> NFCC:C_0603_1608Metric__C17
- C18: footprint Package_SO:TSSOP-28_4.4x9.7mm_P0.65mm -> NFCC:C_0603_1608Metric__C18
- C19: footprint Package_SO:TSSOP-28_4.4x9.7mm_P0.65mm -> NFCC:C_0603_1608Metric__C19
- C20: footprint Package_SO:TSSOP-28_4.4x9.7mm_P0.65mm -> NFCC:C_0603_1608Metric__C20
- C21: footprint Package_SO:TSSOP-28_4.4x9.7mm_P0.65mm -> NFCC:C_0805_2012Metric__C21
- C22: footprint Package_SO:TSSOP-28_4.4x9.7mm_P0.65mm -> NFCC:C_0603_1608Metric__C22
- C23: footprint Package_SO:TSSOP-28_4.4x9.7mm_P0.65mm -> NFCC:C_0805_2012Metric__C23
- C24: footprint Package_SO:TSSOP-28_4.4x9.7mm_P0.65mm -> NFCC:C_0805_2012Metric__C24
- C42: footprint (none) -> NFCC:C_0603_1608Metric__C42
- C43: footprint (none) -> NFCC:C_0603_1608Metric__C43
- C44: footprint (none) -> NFCC:C_0603_1608Metric__C44
- C45: footprint (none) -> NFCC:C_0603_1608Metric__C45
- C46: footprint (none) -> NFCC:C_0603_1608Metric__C46
- C47: footprint (none) -> NFCC:C_0603_1608Metric__C47
- C48: footprint (none) -> NFCC:C_0603_1608Metric__C48
- C49: footprint (none) -> NFCC:C_0603_1608Metric__C49
- C50: footprint (none) -> NFCC:C_0603_1608Metric__C50
- C51: footprint (none) -> NFCC:C_0603_1608Metric__C51
- C52: footprint (none) -> NFCC:C_0603_1608Metric__C52
- C53: footprint (none) -> NFCC:C_0603_1608Metric__C53
- C54: footprint (none) -> NFCC:C_0603_1608Metric__C54
- C55: footprint (none) -> NFCC:C_0603_1608Metric__C55
- C56: footprint (none) -> NFCC:C_0603_1608Metric__C56
- C57: footprint (none) -> NFCC:C_0603_1608Metric__C57
- C58: footprint (none) -> NFCC:C_0603_1608Metric__C58
- C59: footprint (none) -> NFCC:C_0603_1608Metric__C59
- C60: footprint (none) -> NFCC:C_0805_2012Metric__C60
- C61: footprint (none) -> NFCC:C_0603_1608Metric__C61
- C62: footprint (none) -> NFCC:C_0805_2012Metric__C62
- C63: footprint (none) -> NFCC:C_0805_2012Metric__C63
- D1: footprint Package_SON:WSON-8-1EP_6x5mm_P1.27mm_EP3.4x4mm -> NFCC:D_SOD-323__D1
- D2: footprint Package_SON:WSON-8-1EP_6x5mm_P1.27mm_EP3.4x4mm -> NFCC:D_SOD-323__D2
- D3: footprint Package_SO:SOIC-8_3.9x4.9mm_P1.27mm -> NFCC:LED_0603_1608Metric__D3
- D4: footprint Package_SO:SOIC-8_3.9x4.9mm_P1.27mm -> NFCC:LED_0603_1608Metric__D4
- FB1: footprint (none) -> NFCC:L_0805_2012Metric__FB1
- FB2: footprint (none) -> NFCC:L_0805_2012Metric__FB2
- HSE3: footprint (none) -> NFCC:Crystal_SMD_3225-4Pin_3.2x2.5mm__HSE3
- I2C5: value Conn_01x04 -> 53261-0471; footprint Oscillator:Oscillator_SMD_OCXO_ConnorWinfield_OH300 -> NFCC:Molex_PicoBlade_53261-0471_1x04-1MP_P1.25mm_Horizontal__I2C5; symbol Connector_Generic:Conn_01x04 -> NFCC:PicoBlade_4_Grounded_Mounts
- J1: footprint Package_DFN_QFN:WQFN-16-1EP_3x3mm_P0.5mm_EP1.75x1.75mm -> NFCC:USB_Micro-B_Molex_47346-0001__J1
- J2: footprint Package_DFN_QFN:WQFN-16-1EP_3x3mm_P0.5mm_EP1.75x1.75mm -> NFCC:USB_Micro-B_Molex_47346-0001__J2
- J3: footprint (none) -> NFCC:AMASS_XT60-M_1x02_P7.20mm_Vertical__J3
- JP1: footprint Package_SON:WSON-8-1EP_6x5mm_P1.27mm_EP3.4x4mm -> NFCC:SolderJumper-2_P1.3mm_Open_RoundedPad1.0x1.5mm__JP1
- L1: footprint Package_TO_SOT_SMD:SOT-23-6 -> NFCC:L_Bourns_SRN6045TA__L1
- LED13: footprint (none) -> NFCC:LED_0603_1608Metric__LED13
- LED14: footprint (none) -> NFCC:LED_0603_1608Metric__LED14
- LED15: footprint (none) -> NFCC:LED_0603_1608Metric__LED15
- LED16: footprint (none) -> NFCC:LED_0603_1608Metric__LED16
- LED17: footprint (none) -> NFCC:LED_0603_1608Metric__LED17
- LED18: footprint (none) -> NFCC:LED_0603_1608Metric__LED18
- NFCC2: footprint Package_QFP:LQFP-100_14x14mm_P0.5mm -> NFCC:LQFP-100_14x14mm_P0.5mm__NFCC2
- PWM_POW2: footprint (none) -> NFCC:PinHeader_2x08_P2.54mm_Vertical__PWM_POW2
- PWM_SIG2: footprint Oscillator:Oscillator_SMD_OCXO_ConnorWinfield_OH300 -> NFCC:PinHeader_1x08_P2.54mm_Vertical__PWM_SIG2
- R1: footprint Package_DIP:DIP-8_W7.62mm -> NFCC:R_0603_1608Metric__R1
- R2: footprint Package_DIP:DIP-8_W7.62mm -> NFCC:R_0603_1608Metric__R2
- R3: value 52.3k -> 73.2k; footprint Package_DIP:DIP-8_W7.62mm -> NFCC:R_0603_1608Metric__R3
- R35: footprint (none) -> NFCC:R_0603_1608Metric__R35
- R36: footprint (none) -> NFCC:R_0603_1608Metric__R36
- R37: footprint (none) -> NFCC:R_0603_1608Metric__R37
- R38: footprint (none) -> NFCC:R_0603_1608Metric__R38
- R39: footprint (none) -> NFCC:R_0603_1608Metric__R39
- R4: footprint Package_LCC:PLCC-84_29.3x29.3mm_P1.27mm -> NFCC:R_0603_1608Metric__R4
- R40: footprint (none) -> NFCC:R_0603_1608Metric__R40
- R41: footprint (none) -> NFCC:R_0603_1608Metric__R41
- R42: footprint (none) -> NFCC:R_0603_1608Metric__R42
- R43: footprint (none) -> NFCC:R_0603_1608Metric__R43
- R44: footprint (none) -> NFCC:R_0603_1608Metric__R44
- R45: footprint (none) -> NFCC:R_0603_1608Metric__R45
- R46: footprint (none) -> NFCC:R_0603_1608Metric__R46
- R47: footprint (none) -> NFCC:R_0603_1608Metric__R47
- R48: footprint (none) -> NFCC:R_0603_1608Metric__R48
- R49: footprint (none) -> NFCC:R_0603_1608Metric__R49
- R5: footprint Package_LCC:PLCC-84_29.3x29.3mm_P1.27mm -> NFCC:R_0603_1608Metric__R5
- R50: footprint (none) -> NFCC:R_0603_1608Metric__R50
- R51: footprint (none) -> NFCC:R_0603_1608Metric__R51
- R52: footprint (none) -> NFCC:R_0603_1608Metric__R52
- R53: footprint (none) -> NFCC:R_0603_1608Metric__R53
- R54: footprint (none) -> NFCC:R_0603_1608Metric__R54
- R55: footprint (none) -> NFCC:R_0603_1608Metric__R55
- R6: footprint Package_DIP:DIP-8_W7.62mm -> NFCC:R_0603_1608Metric__R6
- R7: footprint Package_DIP:DIP-8_W7.62mm -> NFCC:R_0603_1608Metric__R7
- SW5: footprint (none) -> NFCC:SW_SPST_SKQG_WithoutStem__SW5
- SW6: footprint (none) -> NFCC:SW_SPDT_PCM12__SW6
- SWD2: footprint (none) -> NFCC:PinHeader_2x05_P1.27mm_Vertical__SWD2
- TELEM2: value Conn_01x04 -> 53261-0471; footprint Oscillator:Oscillator_SMD_OCXO_ConnorWinfield_OH300 -> NFCC:Molex_PicoBlade_53261-0471_1x04-1MP_P1.25mm_Horizontal__TELEM2; symbol Connector_Generic:Conn_01x04 -> NFCC:PicoBlade_4_Grounded_Mounts
- TP5: footprint (none) -> NFCC:TestPoint_Pad_D1.5mm__TP5
- TP6: footprint (none) -> NFCC:TestPoint_Pad_D1.5mm__TP6
- U1: footprint Package_SO:SOIC-8_3.9x4.9mm_P1.27mm -> NFCC:SOIC-8_3.9x4.9mm_P1.27mm__U1
- U10: footprint LGA-12_2X2X0P7_STM -> NFCC:LGA-12_2X2X0P7_STM__U10
- U11: footprint SOT-23-5_2P9X1P6_MCH -> NFCC:SOT-23-5_2P9X1P6_MCH__U11
- U12: footprint Package_LGA:Bosch_LGA-16_4.5x3mm_P0.5mm_LayoutBorder7x1y_ClockwisePinNumbering -> NFCC:Bosch_LGA-16_4.5x3mm_P0.5mm_LayoutBorder7x1y_ClockwisePinNumbering__U12
- U2: footprint Package_TO_SOT_SMD:SOT-23-6 -> NFCC:SOT-23-6__U2
- U3: footprint SON_DFN6_3X3_STM -> NFCC:SON_DFN6_3X3_STM__U3
- U7: footprint QFN10_BMP581_BOS -> NFCC:QFN10_BMP581_BOS__U7
- U8: footprint WSON-8_8X6_WIN -> NFCC:WSON-8_8X6_WIN__U8
- U9: footprint Package_SO:TSSOP-28_4.4x9.7mm_P0.65mm -> NFCC:TSSOP-28_4.4x9.7mm_P0.65mm__U9
Connections:
- net +3V3 is gone; now on net +3.3V: SW6.1 (A)
- net GND: now also I2C5.MP (Mount_GND), TELEM2.MP (Mount_GND)
- net VBAT: now also U2.3 (VIN); no longer U2.5 (EN)
- net at R7.1: now also U2.5 (EN); no longer U2.3 (VIN)
Other:
- title: (none) -> NFCC
- moved on the sheet: R7
