File: checks/before-models/NFCC.kicad_pcb (KiCad board)
At the start: 4 copper layers, 90 x 70 mm, 105 parts, among them J1 USB_B_Micro, J2 USB_B_Micro, J3 LiPo Battery, SW5 SW_Push, SW6 SW_SPDT, U1 CH330N, U10 IIS2MDCTR, U11 24CW1280T-I/OT, U12 BMI088, U2 TPS54302, U3 LD39200PU33R, U7 BMP581, U8 W25N01GVZEIG, U9 PCA9685PW

Commit message: Add files via upload
Other:
- board text added: "NFCC REV C"
- board text removed: "NFCC M1:Verity"
Changed lines of the file:
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@@
 		)
 		(embedded_fonts no)
-		(model "${KIPRJMOD}/NFCC.3dshapes/BMP581.step"
-			(offset
-				(xyz 0 0 0)
-			)
-			(scale
-				(xyz 1 1 1)
-			)
-			(rotate
-				(xyz 0 0 0)
-			)
-		)
 	)
 	(footprint "NFCC:R_0603_1608Metric__R44"
@@
 		)
 		(embedded_fonts no)
-		(model "${KIPRJMOD}/NFCC.3dshapes/DFN-6-1EP_3x3mm_P0.95mm_EP1.7x2.6mm.step"
-			(offset
-				(xyz 0 0 0)
-			)
-			(scale
-				(xyz 1 1 1)
-			)
-			(rotate
-				(xyz 0 0 0)
-			)
-		)
 	)
 	(footprint "NFCC:L_0805_2012Metric__FB1"
@@
 		)
 		(embedded_fonts no)
-		(model "${KIPRJMOD}/NFCC.3dshapes/24CW1280T-I_OT.step"
-			(offset
-				(xyz 0 0 0)
-			)
-			(scale
-				(xyz 1 1 1)
-			)
-			(rotate
-				(xyz 0 0 0)
-			)
-		)
 	)
 	(footprint "NFCC:LED_0603_1608Metric__LED15"
@@
 		)
 		(embedded_fonts no)
-		(model "${KIPRJMOD}/NFCC.3dshapes/LGA-12_2x2mm_P0.5mm.step"
-			(offset
-				(xyz 0 0 0)
-			)
-			(scale
-				(xyz 1 1 1)
-			)
-			(rotate
-				(xyz 0 0 0)
-			)
-		)
 	)
 	(footprint "NFCC:R_0603_1608Metric__R36"
@@
 		)
 		(embedded_fonts no)
-		(model "${KIPRJMOD}/NFCC.3dshapes/W25N01GVZEIG.step"
-			(offset
-				(xyz 0 0 0)
-			)
-			(scale
-				(xyz 1 1 1)
-			)
-			(rotate
-				(xyz 0 0 0)
-			)
-		)
 	)
 	(footprint "NFCC:C_0603_1608Metric__C17"
@@
 		)
 	)
-	(gr_text "NFCC M1:Verity"
-		(at 75.5 66.5 0)
+	(gr_text "NFCC REV C"
+		(at 106 76 0)
 		(layer "F.SilkS")
 		(effects
 			(font
-				(size 1.1 1.5)
+				(size 1.1 1.1)
 				(thickness 0.12)
 			)
